File: Hardware/CAD/Sleigh_Controller/Sleigh_Controller_Ornament_2023/Sleigh_Controller_Ornament_2023.kicad_sch (KiCad schematic)
At the start: 2 parts, among them J101 3mm Pitch 5A - 3p, J102 3mm Pitch 5A - 3p

Commit message: PCB Progress
Parts:
- removed J101, J102: 3mm Pitch 5A - 3p, RK_Connector_Terminals:20290303, symbol RK_Connector_Terminals:3mm Pitch 5A - 3p
- added H101, H102, H103: JLC Tooling Hole, RK_Holes:JLC_Tooling, symbol RK_Holes:JLC Tooling Hole
Other:
- added sheet Charlieplexing (Charlieplexing.kicad_sch)
- added sheet Connectors (Connectors.kicad_sch)
- added sheet LEDs (LEDs.kicad_sch)
- added sheet MCU (MCU.kicad_sch)
- added sheet Power (Power.kicad_sch)
