File: Hardware/CAD/Sleigh_Controller/Sleigh_Controller_Ornament_2023/LEDs.kicad_sch (KiCad schematic)
At the start: 66 parts, among them U601 74HC14D,653

Commit message: pcb progress continued
Parts:
- removed C104: 0.1uF 16V 0402, Capacitor_SMD:C_0402_1005Metric, symbol Device:C_Small
- removed D615: WS2812B-2020, RK_LED_SMD:LED_WS2812B-2020, symbol RK_LED:WS2812B-2020
- removed R203: 10k 1% 0402, Resistor_SMD:R_0402_1005Metric, symbol Device:R_Small_US
- removed R203: 33 1% 0402, Resistor_SMD:R_0402_1005Metric, symbol Device:R_Small_US
- added R203: 10k 1% 0402, Resistor_SMD:R_0402_1005Metric, symbol Device:R_Small_US
Connections:
- net GND: now also R203.2
- net at R203.1: now also R203.1
