File: Hardware/CAD/Sleigh_Controller/Sleigh_Controller_Ornament_2023/Sleigh_Controller_Ornament_2023.kicad_pcb (KiCad board)
At the start: 2 copper layers, 99.8 x 99.6 mm, 1 part

Commit message: PCB Progress
Parts:
- removed REF**: ESP32-WROVER-E, RK_MCU_Modules:ESP32-WROVER-E
- added C201: 10uF 10V 0603, Capacitor_SMD:C_0603_1608Metric, B.Cu at (151.6, 98.8)
- added C202: 10uF 10V 0603, Capacitor_SMD:C_0603_1608Metric, B.Cu at (153.4, 98.8)
- added C205: 0.1uF 16V 0402, Capacitor_SMD:C_0402_1005Metric, B.Cu at (124.0, 61.0)
- added C206: 0.1uF 16V 0402, Capacitor_SMD:C_0402_1005Metric, B.Cu at (130.6, 72.3)
- added C207: 10uF 10V 0603, Capacitor_SMD:C_0603_1608Metric, B.Cu at (123.9, 63.0)
- added C301: 10uF 10V 0603, Capacitor_SMD:C_0603_1608Metric, B.Cu at (124.7, 65.4)
- added C302: 0.1uF 16V 0402, Capacitor_SMD:C_0402_1005Metric, B.Cu at (128.6, 69.7)
- added C303: 0.1uF 16V 0402, Capacitor_SMD:C_0402_1005Metric, B.Cu at (124.6, 77.2)
- added C305: 0.1uF 16V 0402, Capacitor_SMD:C_0402_1005Metric, B.Cu at (117.1, 81.9)
- added C306: 0.1uF 16V 0402, Capacitor_SMD:C_0402_1005Metric, B.Cu at (121.2, 81.9)
- added C308: 0.1uF 16V 0402, Capacitor_SMD:C_0402_1005Metric, B.Cu at (128.7, 75.3)
- added C309: 10uF 10V 0603, Capacitor_SMD:C_0603_1608Metric, B.Cu at (129.3, 76.7)
- added C310: 10uF 10V 0603, Capacitor_SMD:C_0603_1608Metric, B.Cu at (132.7, 47.6)
- added C311: 0.1uF 16V 0402, Capacitor_SMD:C_0402_1005Metric, B.Cu at (130.3, 47.9)
- added C312: 0.1uF 16V 0402, Capacitor_SMD:C_0402_1005Metric, B.Cu at (137.2, 47.2)
- added C313: 10uF 10V 0603, Capacitor_SMD:C_0603_1608Metric, B.Cu at (139.1, 48.0)
- added C401: 10uF 10V 0603, Capacitor_SMD:C_0603_1608Metric, B.Cu at (148.7, 65.8)
- added C402: 0.1uF 16V 0402, Capacitor_SMD:C_0402_1005Metric, B.Cu at (148.3, 63.9)
- added C501: 0.1uF 16V 0402, Capacitor_SMD:C_0402_1005Metric, B.Cu at (169.2, 98.8)
- added C502: 0.1uF 16V 0402, Capacitor_SMD:C_0402_1005Metric, B.Cu at (167.2, 98.8)
- added C503: 0.1uF 16V 0402, Capacitor_SMD:C_0402_1005Metric, B.Cu at (143.9, 68.8)
- added C504: 0.1uF 16V 0402, Capacitor_SMD:C_0402_1005Metric, B.Cu at (146.6, 71.0)
- added C505: 0.1uF 16V 0402, Capacitor_SMD:C_0402_1005Metric, B.Cu at (139.2, 70.0)
- added C506: 0.1uF 16V 0402, Capacitor_SMD:C_0402_1005Metric, B.Cu at (135.5, 70.2)
- added C601: 0.1uF 16V 0402, Capacitor_SMD:C_0402_1005Metric, B.Cu at (131.2, 80.7)
- added C602: 0.1uF 16V 0402, Capacitor_SMD:C_0402_1005Metric, B.Cu at (143.6, 86.1)
- added C603: 0.1uF 16V 0402, Capacitor_SMD:C_0402_1005Metric, B.Cu at (143.6, 82.0)
- added C604: 0.1uF 16V 0402, Capacitor_SMD:C_0402_1005Metric, B.Cu at (114.6, 88.8)
- added C605: 0.1uF 16V 0402, Capacitor_SMD:C_0402_1005Metric, B.Cu at (114.4, 96.0)
- added C606: 0.1uF 16V 0402, Capacitor_SMD:C_0402_1005Metric, B.Cu at (120.1, 107.2)
- added C607: 0.1uF 16V 0402, Capacitor_SMD:C_0402_1005Metric, B.Cu at (126.5, 114.3)
- added C608: 0.1uF 16V 0402, Capacitor_SMD:C_0402_1005Metric, B.Cu at (121.9, 123.7)
- added C609: 0.1uF 16V 0402, Capacitor_SMD:C_0402_1005Metric, B.Cu at (127.0, 128.9)
- added C610: 0.1uF 16V 0402, Capacitor_SMD:C_0402_1005Metric, B.Cu at (140.1, 128.9)
- added C611: 0.1uF 16V 0402, Capacitor_SMD:C_0402_1005Metric, B.Cu at (155.7, 128.9)
- added C612: 0.1uF 16V 0402, Capacitor_SMD:C_0402_1005Metric, B.Cu at (169.3, 128.9)
- added C613: 0.1uF 16V 0402, Capacitor_SMD:C_0402_1005Metric, B.Cu at (183.8, 127.5)
- added C614: 0.1uF 16V 0402, Capacitor_SMD:C_0402_1005Metric, B.Cu at (24.4, 63.1)
- added C615: 0.1uF 16V 0402, Capacitor_SMD:C_0402_1005Metric, B.Cu at (24.4, 65.1)
- added C616: 0.1uF 16V 0402, Capacitor_SMD:C_0402_1005Metric, B.Cu at (21.6, 53.3)
- added C617: 0.1uF 16V 0402, Capacitor_SMD:C_0402_1005Metric, B.Cu at (21.6, 55.2)
- added C618: 0.1uF 16V 0402, Capacitor_SMD:C_0402_1005Metric, B.Cu at (21.6, 57.2)
- added C619: 0.1uF 16V 0402, Capacitor_SMD:C_0402_1005Metric, B.Cu at (21.6, 59.2)
- added D201: SRV05-4, Package_TO_SOT_SMD:SOT-23-6, B.Cu at (127.2, 60.0)
- added D301: 350mA 28V, Diode_SMD:D_SOD-323, B.Cu at (119.2, 69.3)
- added D302: 350mA 28V, Diode_SMD:D_SOD-323, B.Cu at (119.2, 67.1)
- added D501: 350mA 28V, Diode_SMD:D_SOD-323, B.Cu at (146.6, 75.2)
- added D502: 350mA 28V, Diode_SMD:D_SOD-323, B.Cu at (171.3, 81.2)
- added D503: 350mA 28V, Diode_SMD:D_SOD-323, B.Cu at (167.6, 81.2)
- added D504: 350mA 28V, Diode_SMD:D_SOD-323, B.Cu at (144.3, 75.2)
- added D505: 350mA 28V, Diode_SMD:D_SOD-323, B.Cu at (146.6, 78.8)
- added D506: 350mA 28V, Diode_SMD:D_SOD-323, B.Cu at (152.1, 65.7)
- added D507: 350mA 28V, Diode_SMD:D_SOD-323, B.Cu at (173.2, 77.9)
- added D508: 350mA 28V, Diode_SMD:D_SOD-323, B.Cu at (174.9, 81.2)
- added D509: 350mA 28V, Diode_SMD:D_SOD-323, B.Cu at (152.1, 63.5)
- added D510: 350mA 28V, Diode_SMD:D_SOD-323, B.Cu at (176.0, 78.4)
- added D511: 350mA 28V, Diode_SMD:D_SOD-323, B.Cu at (152.2, 61.3)
- added D601: WS2812B-2020, RK_LED_SMD:LED_WS2812B-2020, B.Cu at (143.2, 80.0)
- added D602: WS2812B-2020, RK_LED_SMD:LED_WS2812B-2020, B.Cu at (143.2, 84.1)
- added D603: WS2812B-2020, RK_LED_SMD:LED_WS2812B-2020, B.Cu at (112.6, 89.3)
- added D604: WS2812B-2020, RK_LED_SMD:LED_WS2812B-2020, B.Cu at (114.3, 98.7)
- added D605: WS2812B-2020, RK_LED_SMD:LED_WS2812B-2020, B.Cu at (121.8, 109.1)
- added D606: WS2812B-2020, RK_LED_SMD:LED_WS2812B-2020, B.Cu at (126.5, 117.1)
- added D607: WS2812B-2020, RK_LED_SMD:LED_WS2812B-2020, B.Cu at (120.1, 125.7)
- added D608: WS2812B-2020, RK_LED_SMD:LED_WS2812B-2020, B.Cu at (129.6, 129.2)
- added D609: WS2812B-2020, RK_LED_SMD:LED_WS2812B-2020, B.Cu at (142.7, 129.1)
- added D610: WS2812B-2020, RK_LED_SMD:LED_WS2812B-2020, B.Cu at (158.3, 129.2)
- added D611: WS2812B-2020, RK_LED_SMD:LED_WS2812B-2020, B.Cu at (172.0, 129.1)
- added D612: WS2812B-2020, RK_LED_SMD:LED_WS2812B-2020, B.Cu at (186.1, 126.0)
- added D613: WS2812B-2020, RK_LED_SMD:LED_WS2812B-2020, B.Cu at (30.8, 54.0)
- added D614: WS2812B-2020, RK_LED_SMD:LED_WS2812B-2020, B.Cu at (30.8, 57.6)
- added D615: WS2812B-2020, RK_LED_SMD:LED_WS2812B-2020, B.Cu at (30.8, 61.1)
- added D616: WS2812B-2020, RK_LED_SMD:LED_WS2812B-2020, B.Cu at (30.8, 64.7)
- added D617: WS2812B-2020, RK_LED_SMD:LED_WS2812B-2020, B.Cu at (30.8, 68.2)
- added D618: WS2812B-2020, RK_LED_SMD:LED_WS2812B-2020, B.Cu at (30.8, 71.8)
- added H101: JLC Tooling Hole, RK_Holes:JLC_Tooling, F.Cu at (134.1, 34.0)
- added H102: JLC Tooling Hole, RK_Holes:JLC_Tooling, F.Cu at (184.0, 77.7)
- added H103: JLC Tooling Hole, RK_Holes:JLC_Tooling, F.Cu at (116.8, 107.2)
- added J201: 3mm Pitch 5A - 3p, RK_Connector_Terminals:20290303, B.Cu at (143.3, 96.2)
- added J202: 3mm Pitch 5A - 3p, RK_Connector_Terminals:20290303, B.Cu at (158.3, 90.2)
- added J203: GT-USB-7047C, RK_Connector_USB:GT-USB-7047C, B.Cu at (121.8, 54.2)
- added Q301: 20V 28mOhm, Package_TO_SOT_SMD:SOT-23-3, B.Cu at (123.2, 70.4)
- added R201: 5.1k 1% 0402, Resistor_SMD:R_0402_1005Metric, B.Cu at (118.1, 62.4)
- added R202: 5.1k 1% 0402, Resistor_SMD:R_0402_1005Metric, B.Cu at (120.0, 65.0)
- added R301: 5.1k 1% 0402, Resistor_SMD:R_0402_1005Metric, B.Cu at (117.9, 71.8)
- added R302: 5.1k 1% 0402, Resistor_SMD:R_0402_1005Metric, B.Cu at (120.4, 71.8)
- added R303: 0ohm 0805, Resistor_SMD:R_0805_2012Metric, B.Cu at (128.2, 67.9)
- added R304: 5.1k 1% 0402, Resistor_SMD:R_0402_1005Metric, B.Cu at (125.6, 71.6)
- added R305: 4.7k 1% 0402, Resistor_SMD:R_0402_1005Metric, B.Cu at (113.7, 77.2)
- added R306: 20k 1% 0805, Resistor_SMD:R_0805_2012Metric, B.Cu at (119.1, 85.5)
- added R307: 4.7k 1% 1206, Resistor_SMD:R_1206_3216Metric, B.Cu at (126.5, 77.2)
- added R308: 5.1k 1% 0402, Resistor_SMD:R_0402_1005Metric, B.Cu at (119.1, 82.4)
- added R309: 10k 1% 0402, Resistor_SMD:R_0402_1005Metric, B.Cu at (125.6, 73.8)
- added R310: 150k 1% 0402, Resistor_SMD:R_0402_1005Metric, B.Cu at (113.7, 79.6)
- added R311: 150k 1% 0402, Resistor_SMD:R_0402_1005Metric, B.Cu at (125.0, 80.1)
- added R312: 8.2k 1% 0402, Resistor_SMD:R_0402_1005Metric, B.Cu at (124.5, 73.8)
- added R313: 0ohm 1206, Resistor_SMD:R_1206_3216Metric, B.Cu at (129.4, 86.8)
- added R314: 0ohm 1206, Resistor_SMD:R_1206_3216Metric, B.Cu at (116.5, 87.6)
- added R315: 10k 1% 0402, Resistor_SMD:R_0402_1005Metric, B.Cu at (123.2, 67.6)
- added R316: 33 1% 0402, Resistor_SMD:R_0402_1005Metric, B.Cu at (115.2, 82.4)
- added R317: 33 1% 0402, Resistor_SMD:R_0402_1005Metric, B.Cu at (123.1, 82.4)
- added R402: 33 1% 0805, Resistor_SMD:R_0805_2012Metric, B.Cu at (130.3, 58.2)
- added R403: 33 1% 0805, Resistor_SMD:R_0805_2012Metric, B.Cu at (128.9, 56.8)
- added R404: 33 1% 0402, Resistor_SMD:R_0402_1005Metric, B.Cu at (133.2, 63.6)
- added R405: 33 1% 0402, Resistor_SMD:R_0402_1005Metric, B.Cu at (135.0, 65.4)
- added R406: 33 1% 0402, Resistor_SMD:R_0402_1005Metric, B.Cu at (134.1, 64.5)
- added R407: 10k 1% 0402, Resistor_SMD:R_0402_1005Metric, B.Cu at (145.4, 67.4)
- added R408: 10k 1% 0402, Resistor_SMD:R_0402_1005Metric, B.Cu at (146.3, 66.5)
- added R409: 10k 1% 0402, Resistor_SMD:R_0402_1005Metric, B.Cu at (132.3, 62.7)
- added R410: 10k 1% 0402, Resistor_SMD:R_0402_1005Metric, B.Cu at (131.4, 61.8)
- added R501: 510k 1% 0402, Resistor_SMD:R_0402_1005Metric, B.Cu at (142.3, 69.7)
- added R502: 510k 1% 0402, Resistor_SMD:R_0402_1005Metric, B.Cu at (145.4, 71.0)
- added R503: 510k 1% 0402, Resistor_SMD:R_0402_1005Metric, B.Cu at (137.3, 67.2)
- added R504: 510k 1% 0402, Resistor_SMD:R_0402_1005Metric, B.Cu at (135.7, 66.4)
- added R505: 1k 1% 0402, Resistor_SMD:R_0402_1005Metric, B.Cu at (143.8, 70.6)
- added R506: 1k 1% 0402, Resistor_SMD:R_0402_1005Metric, B.Cu at (144.1, 72.3)
- added R507: 1k 1% 0402, Resistor_SMD:R_0402_1005Metric, B.Cu at (137.5, 69.1)
- added R508: 1k 1% 0402, Resistor_SMD:R_0402_1005Metric, B.Cu at (135.9, 68.6)
- added R509: 1k 1% 0402, Resistor_SMD:R_0402_1005Metric, B.Cu at (166.6, 100.5)
- added R510: 1k 1% 0402, Resistor_SMD:R_0402_1005Metric, B.Cu at (169.7, 100.5)
- added R511: 1k 1% 0402, Resistor_SMD:R_0402_1005Metric, B.Cu at (146.1, 69.2)
- added R512: 1k 1% 0402, Resistor_SMD:R_0402_1005Metric, B.Cu at (145.9, 72.8)
- added R513: 1k 1% 0402, Resistor_SMD:R_0402_1005Metric, B.Cu at (140.6, 71.1)
- added R514: 1k 1% 0402, Resistor_SMD:R_0402_1005Metric, B.Cu at (137.5, 70.8)
- added R601: 0 1% 0402, Resistor_SMD:R_0402_1005Metric, B.Cu at (133.6, 72.8)
- added R602: 0 1% 0402, Resistor_SMD:R_0402_1005Metric, B.Cu at (134.7, 81.9)
- added R603: 0 1% 0402, Resistor_SMD:R_0402_1005Metric, B.Cu at (136.1, 72.8)
- added R604: 0 1% 0402, Resistor_SMD:R_0402_1005Metric, B.Cu at (137.3, 81.9)
- added R605: 0 1% 0402, Resistor_SMD:R_0402_1005Metric, B.Cu at (138.6, 72.8)
- added R606: 0 1% 0402, Resistor_SMD:R_0402_1005Metric, B.Cu at (139.8, 81.9)
- added R607: 33 1% 0805, Resistor_SMD:R_0805_2012Metric, B.Cu at (137.3, 84.3)
- added R608: 33 1% 0805, Resistor_SMD:R_0805_2012Metric, B.Cu at (139.8, 84.3)
- added R609: 33 1% 0805, Resistor_SMD:R_0805_2012Metric, B.Cu at (147.1, 81.8)
- added R610: 33 1% 0805, Resistor_SMD:R_0805_2012Metric, B.Cu at (147.1, 84.3)
- added R611: 33 1% 0402, Resistor_SMD:R_0402_1005Metric, B.Cu at (135.4, 83.8)
- added R612: 33 1% 0402, Resistor_SMD:R_0402_1005Metric, B.Cu at (113.2, 91.9)
- added R613: 33 1% 0402, Resistor_SMD:R_0402_1005Metric, B.Cu at (114.8, 101.7)
- added R614: 33 1% 0402, Resistor_SMD:R_0402_1005Metric, B.Cu at (124.2, 112.0)
- added R615: 33 1% 0402, Resistor_SMD:R_0402_1005Metric, B.Cu at (125.1, 119.9)
- added R616: 33 1% 0402, Resistor_SMD:R_0402_1005Metric, B.Cu at (118.0, 128.0)
- added R617: 33 1% 0402, Resistor_SMD:R_0402_1005Metric, B.Cu at (132.8, 129.4)
- added R618: 33 1% 0402, Resistor_SMD:R_0402_1005Metric, B.Cu at (145.9, 129.4)
- added R619: 33 1% 0402, Resistor_SMD:R_0402_1005Metric, B.Cu at (161.5, 129.4)
- added R620: 33 1% 0402, Resistor_SMD:R_0402_1005Metric, B.Cu at (175.1, 129.4)
- added R621: 33 1% 0402, Resistor_SMD:R_0402_1005Metric, B.Cu at (185.0, 123.1)
- added R622: 33 1% 0402, Resistor_SMD:R_0402_1005Metric, B.Cu at (21.5, 73.0)
- added R623: 33 1% 0402, Resistor_SMD:R_0402_1005Metric, B.Cu at (21.5, 75.0)
- added R624: 33 1% 0402, Resistor_SMD:R_0402_1005Metric, B.Cu at (21.5, 77.0)
- added R625: 33 1% 0402, Resistor_SMD:R_0402_1005Metric, B.Cu at (18.6, 67.1)
- added R626: 33 1% 0402, Resistor_SMD:R_0402_1005Metric, B.Cu at (18.6, 69.0)
- added R627: 33 1% 0402, Resistor_SMD:R_0402_1005Metric, B.Cu at (18.6, 71.0)
- added R628: 10k 1% 0402, Resistor_SMD:R_0402_1005Metric, B.Cu at (18.6, 73.0)
- added SW501: SW_DIP_x05_alt, RK_Switches:EM-05KP, B.Cu at (160.7, 110.2)
- added SW502: SW_DIP_x08, RK_Switches:SMXS-08K-TP, B.Cu at (159.5, 73.5)
- added U301: LMV324, Package_SO:SO-14_3.9x8.65mm_P1.27mm, B.Cu at (119.1, 77.3)
- added U302: MT9700, Package_TO_SOT_SMD:SOT-23-5, B.Cu at (128.1, 72.5)
- added U303: AMS1117-3.3, Package_TO_SOT_SMD:SOT-223-3_TabPin2, B.Cu at (133.8, 42.1)
- added U401: ESP32-C3-MINI-1-N4, RK_MCU_Modules:ESP32-C3-MINI-1-N4, B.Cu at (140.5, 60.0)
- added U601: 74HC14D,653, Package_SO:SO-14_3.9x8.65mm_P1.27mm, B.Cu at (136.7, 77.3)
Routing:
- net GND: track 0.00 -> 213.6 mm, vias 0 -> 75
- net VDD_3V3: track 0.00 -> 128.6 mm
- net VLED_5V0: track 0.00 -> 109.8 mm
- net Net-(D511-A2): track 0.00 -> 97.5 mm
- net /Charlieplexing/CMUX_2_SW_3V3: track 0.00 -> 81.1 mm
- net /Charlieplexing/MCU_BOOTMODE_3V3: track 0.00 -> 77.7 mm
- net /Charlieplexing/MCU_EN_3V3: track 0.00 -> 76.4 mm
- net /Charlieplexing/CMUX_3_SW_3V3: track 0.00 -> 73.2 mm
- net /Charlieplexing/CMUX_1_SW_3V3: track 0.00 -> 68.1 mm
- net Net-(D510-A2): track 0.00 -> 61.0 mm
- net Net-(D508-A2): track 0.00 -> 60.9 mm
- net /Power/LDO_IN_5V0: track 0.00 -> 40.0 mm
- net /Connectors/LED_UP_OUT_5V0: track 0.00 -> 32.0 mm
- net Net-(D302-A2): track 0.00 -> 30.7 mm
- net Net-(D603-DIN): track 0.00 -> 25.4 mm
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- added copper zone on B.Cu, net /Power/LDO_IN_5V0
- added copper zone on F.Cu, net GND
- added copper zone on B.Cu, net VBUS_5V0
- added copper zone on B.Cu, net VDD_3V3
- added copper zone on B.Cu, net VLED_5V0
- added copper zone on B.Cu, net VLED_JUMP_5V0
- removed copper zone on F.Cu, net (none)

Commit message: pcb progress continued
Parts:
- removed C616: 0.1uF 16V 0402, Capacitor_SMD:C_0402_1005Metric
- removed D615: WS2812B-2020, RK_LED_SMD:LED_WS2812B-2020
- removed R628: 10k 1% 0402, Resistor_SMD:R_0402_1005Metric
- R624: value 33 1% 0402 -> 10k 1% 0402
- moved C619 175.2 mm to (191.4, 102.4), turned to 0 degrees
- moved R627 175.2 mm to (191.9, 96.4), turned to -90 degrees
- moved R626 174.7 mm to (192.3, 87.6), turned to -90 degrees
- moved C618 174.2 mm to (191.9, 93.6), turned to 0 degrees
- moved R625 173.9 mm to (192.0, 79.0), turned to -45 degrees
- moved C617 173.3 mm to (192.3, 85.0), turned to 0 degrees
- moved R623 172.5 mm to (190.6, 108.6), turned to -135 degrees
- moved R624 168.0 mm to (189.5, 79.2), turned to -90 degrees
- moved C615 167.9 mm to (185.7, 112.0), turned to -90 degrees
- moved C614 166.9 mm to (181.5, 119.5), turned to 0 degrees
- moved D614 166.0 mm to (188.0, 110.9)
- moved D618 163.3 mm to (191.7, 99.7), turned to -135 degrees
- moved D617 162.9 mm to (192.1, 90.9), turned to -135 degrees
- moved D616 162.7 mm to (192.5, 82.3), turned to -135 degrees
- moved R622 162.4 mm to (178.4, 114.7), turned to -90 degrees
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Connections:
- R624 pad 2: Net-(D615-DOUT) -> GND
- R625 pad 1: Net-(D615-DIN) -> Net-(R624-Pad1)
Routing:
- net Net-(D510-A2): track 61.0 -> 47.4 mm
- net Net-(D508-A2): track 60.9 -> 47.6 mm
- net Net-(D511-A2): track 97.5 -> 84.2 mm
- net Net-(D608-DIN): track 0.00 -> 11.2 mm
- net Net-(D610-DIN): track 0.00 -> 11.1 mm
- net Net-(D612-DIN): track 0.00 -> 10.6 mm
- net Net-(D614-DIN): track 0.00 -> 9.76 mm
- net GND: track 213.6 -> 222.8 mm, vias 75 -> 203
- net Net-(D611-DIN): track 0.00 -> 9.13 mm
- net Net-(D609-DIN): track 0.00 -> 8.60 mm
- net Net-(D618-DIN): track 0.00 -> 7.64 mm
- net Net-(D613-DIN): track 0.00 -> 6.77 mm
- net Net-(D617-DIN): track 0.00 -> 3.92 mm
- net Net-(D616-DIN): track 0.00 -> 3.80 mm
- net /Connectors/USB_DM: track 8.31 -> 11.1 mm
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- added copper zone on B.Cu, net GND
- added copper zone on In1.Cu, net GND
- added copper zone on In2.Cu, net GND
Other:
- copper layers 2 -> 4
- board text added: "0b000"
- board text added: "1"
- board text added: "2"
- board text added: "3"
- board text added: "4"
- board text added: "5"
- board text added: "6"
- board text added: "7"
- board text added: "8"
- board text added: "BOOTMODE"
- board text added: "Configure House Orientations"
- board text added: "House #:"
- board text added: "OFF"
- board text added: "OFF: Horizontal"
- board text added: "ON"
- board text added: "ON: Vertical"
- board text added: "QTY of Houses"
- board text added: "RESET"
